File: Hardware/Electronics/kicad_RCJ/kicad_RCJ.kicad_sch (KiCad schematic)
At the start: 79 parts, among them J1 Raspberry_Pi_2_3, J10 Conn_01x04_M1_extra, J11 Conn_01x04_M2_extra, J12 Conn_01x04_M3_extra, J13 Conn_01x04_M4_extra, J14 Conn_01x06_teensy_left_extra, J15 Conn_01x04_teensy_right_extra, J16 Conn_01x07_IO_expander_extra, J17 Conn_02x03_I2C, J18 Conn_02x05_3V3_GND, J19 Conn_02x05_5V_GND, J2 Conn_01x06_IMU_extra, J20 Conn_01x06_BNO085_extra, J21 Conn_01x06_ISM20948_extra, J22 Conn_01x02_LSM5DSOX_LIS3MDL_e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, J3 Conn_01x02_colsens_interrupt, J4 Conn_01x02_5V, J5 Conn_01x02_3V3, J6 Conn_01x02_I2C1, J7 Conn_01x01_LOP, J8 Conn_01x03_IO_expander_interr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, J9 Conn_01x06_LED, M5 Servo1, M6 Servo2, U1 DRV8874, U12 VL53L0/1X, U13 VL53L0/1X, U14 VL53L0/1X, U15 VL53L0/1X, U16 VL53L0/1X, U17 VL53L0/1X, U18 VL53L0/1X, U2 DRV8874, U20 BNO085, U21 ICM20948, U22 LSM6DSOX+LIS3MDL, U23 TCS34725, U24 APDS9960, U25 VL53L0/1X, U3 DRV8874, U4 DRV8874

Commit message: refined PCB layout and resolved some footprint issues
Parts:
- J9: footprint Connector_PinSocket_2.54mm:PinSocket_1x01_P2.54mm_Vertical -> Connector_PinSocket_2.54mm:PinSocket_1x06_P2.54mm_Vertical
- R1, R10, R12, R13, R14, R2, R3, R4, R6, R8: footprint (none) -> Resistor_THT:R_Axial_DIN0207_L6.3mm_D2.5mm_P7.62mm_Horizontal
- U12, U13, U14, U15, U16, U17, U18, U25: footprint Connector_JST:JST_XH_B6B-XH-A_1x06_P2.50mm_Vertical -> RCJ2024_kicad_footprints:VL53L0X_VL53L1X_connector; symbol RCJ_parts:VL53L0X/VL53L1X -> RCJ_parts:VL53L0X/VL53L1X_NC
Changed lines of the file:
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@@
       (effects (font (size 1.27 1.27)) (justify left))
     )
-    (property "Footprint" "Connector_PinSocket_2.54mm:PinSocket_1x01_P2.54mm_Vertical" (at 386.08 236.22 0)
+    (property "Footprint" "Connector_PinSocket_2.54mm:PinSocket_1x06_P2.54mm_Vertical" (at 386.08 236.22 0)
       (effects (font (size 1.27 1.27)) hide)
     )
@@
     )
   )
-  (symbol (lib_id "RCJ_parts:VL53L0X/VL53L1X") (at 394.97 83.82 0) (unit 1)
+  (symbol (lib_id "RCJ_parts:VL53L0X/VL53L1X_NC") (at 394.97 83.82 0) (unit 1)
     (in_bom yes) (on_board yes) (dnp no)
     (property "Reference" "U18" (at 400.05 91.44 0)
@@
       (effects (font (size 1.27 1.27)))
     )
-    (property "Footprint" "Connector_JST:JST_XH_B6B-XH-A_1x06_P2.50mm_Vertical" (at 394.97 83.82 0)
+    (property "Footprint" "RCJ2024_kicad_footprints:VL53L0X_VL53L1X_connector" (at 394.97 78.74 0)
       (effects (font (size 1.27 1.27)) hide)
     )
@@
       (effects (font (size 1.27 1.27)) hide)
     )
-    (pin "1")
     (pin "2")
     (pin "3")
@@
     (pin "5")
     (pin "6")
-    (pin "7")
     (instances
       (project "kicad_RCJ"
@@
       (effects (font (size 1.27 1.27)) (justify left))
     )
-    (property "Footprint" "" (at 43.942 226.06 90)
+    (property "Footprint" "Resistor_THT:R_Axial_DIN0207_L6.3mm_D2.5mm_P7.62mm_Horizontal" (at 43.942 226.06 90)
       (effects (font (size 1.27 1.27)) hide)
     )
@@
       (effects (font (size 1.27 1.27)) (justify left))
     )
-    (property "Footprint" "" (at 43.942 236.22 90)
+    (property "Footprint" "Resistor_THT:R_Axial_DIN0207_L6.3mm_D2.5mm_P7.62mm_Horizontal" (at 43.942 236.22 90)
       (effects (font (size 1.27 1.27)) hide)
     )
@@
       (effects (font (size 1.27 1.27)) (justify left))
     )
-    (property "Footprint" "" (at 221.742 265.43 90)
+    (property "Footprint" "Resistor_THT:R_Axial_DIN0207_L6.3mm_D2.5mm_P7.62mm_Horizontal" (at 221.742 265.43 90)
       (effects (font (size 1.27 1.27)) hide)
     )
@@
       (effects (font (size 1.27 1.27)) (justify left))
     )
-    (property "Footprint" "" (at 243.332 135.89 90)
+    (property "Footprint" "Resistor_THT:R_Axial_DIN0207_L6.3mm_D2.5mm_P7.62mm_Horizontal" (at 243.332 135.89 90)
       (effects (font (size 1.27 1.27)) hide)
     )
@@
       (effects (font (size 1.27 1.27)) (justify left))
     )
-    (property "Footprint" "" (at 216.662 135.89 90)
+    (property "Footprint" "Resistor_THT:R_Axial_DIN0207_L6.3mm_D2.5mm_P7.62mm_Horizontal" (at 216.662 135.89 90)
       (effects (font (size 1.27 1.27)) hide)
     )
@@
       (effects (font (size 1.27 1.27)) (justify left))
     )
-    (property "Footprint" "" (at 257.302 135.89 90)
+    (property "Footprint" "Resistor_THT:R_Axial_DIN0207_L6.3mm_D2.5mm_P7.62mm_Horizontal" (at 257.302 135.89 90)
       (effects (font (size 1.27 1.27)) hide)
     )
@@
     )
   )
-  (symbol (lib_id "RCJ_parts:VL53L0X/VL53L1X") (at 394.97 62.23 0) (unit 1)
+  (symbol (lib_id "RCJ_parts:VL53L0X/VL53L1X_NC") (at 394.97 62.23 0) (unit 1)
     (in_bom yes) (on_board yes) (dnp no)
     (property "Reference" "U17" (at 400.05 69.85 0)
@@
       (effects (font (size 1.27 1.27)))
     )
-    (property "Footprint" "Connector_JST:JST_XH_B6B-XH-A_1x06_P2.50mm_Vertical" (at 394.97 62.23 0)
+    (property "Footprint" "RCJ2024_kicad_footprints:VL53L0X_VL53L1X_connector" (at 394.97 57.15 0)
       (effects (font (size 1.27 1.27)) hide)
     )
@@
       (effects (font (size 1.27 1.27)) hide)
     )
-    (pin "1")
     (pin "2")
     (pin "3")
@@
     (pin "5")
     (pin "6")
-    (pin "7")
     (instances
       (project "kicad_RCJ"
@@
       (effects (font (size 1.27 1.27)) (justify left))
     )
-    (property "Footprint" "" (at 229.362 265.43 90)
+    (property "Footprint" "Resistor_THT:R_Axial_DIN0207_L6.3mm_D2.5mm_P7.62mm_Horizontal" (at 229.362 265.43 90)
       (effects (font (size 1.27 1.27)) hide)
     )
@@
       (effects (font (size 1.27 1.27)) (justify left))
     )
-    (property "Footprint" "" (at 248.412 265.43 90)
+    (property "Footprint" "Resistor_THT:R_Axial_DIN0207_L6.3mm_D2.5mm_P7.62mm_Horizontal" (at 248.412 265.43 90)
       (effects (font (size 1.27 1.27)) hide)
     )
@@
     )
   )
-  (symbol (lib_id "RCJ_parts:VL53L0X/VL53L1X") (at 394.97 19.05 0) (unit 1)
+  (symbol (lib_id "RCJ_parts:VL53L0X/VL53L1X_NC") (at 394.97 19.05 0) (unit 1)
     (in_bom yes) (on_board yes) (dnp no)
     (property "Reference" "U15" (at 400.05 26.67 0)
@@
       (effects (font (size 1.27 1.27)))
     )
-    (property "Footprint" "Connector_JST:JST_XH_B6B-XH-A_1x06_P2.50mm_Vertical" (at 394.97 19.05 0)
+    (property "Footprint" "RCJ2024_kicad_footprints:VL53L0X_VL53L1X_connector" (at 394.97 13.97 0)
       (effects (font (size 1.27 1.27)) hide)
     )
@@
       (effects (font (size 1.27 1.27)) hide)
     )
-    (pin "1")
     (pin "2")
     (pin "3")
@@
     (pin "5")
     (pin "6")
-    (pin "7")
     (instances
       (project "kicad_RCJ"
@@
     )
   )
-  (symbol (lib_id "RCJ_parts:VL53L0X/VL53L1X") (at 364.49 87.63 0) (unit 1)
+  (symbol (lib_id "RCJ_parts:VL53L0X/VL53L1X_NC") (at 364.49 87.63 0) (unit 1)
     (in_bom yes) (on_board yes) (dnp no)
     (property "Reference" "U25" (at 369.57 95.25 0)
@@
       (effects (font (size 1.27 1.27)))
     )
-    (property "Footprint" "Connector_JST:JST_XH_B6B-XH-A_1x06_P2.50mm_Vertical" (at 364.49 87.63 0)
+    (property "Footprint" "RCJ2024_kicad_footprints:VL53L0X_VL53L1X_connector" (at 364.49 82.55 0)
       (effects (font (size 1.27 1.27)) hide)
     )
@@
       (effects (font (size 1.27 1.27)) hide)
     )
-    (pin "1")
     (pin "2")
     (pin "3")
@@
     (pin "5")
     (pin "6")
-    (pin "7")
     (instances
       (project "kicad_RCJ"
@@
     )
   )
-  (symbol (lib_id "RCJ_parts:VL53L0X/VL53L1X") (at 364.49 40.64 0) (unit 1)
+  (symbol (lib_id "RCJ_parts:VL53L0X/VL53L1X_NC") (at 364.49 40.64 0) (unit 1)
     (in_bom yes) (on_board yes) (dnp no)
     (property "Reference" "U13" (at 369.57 48.26 0)
@@
       (effects (font (size 1.27 1.27)))
     )
-    (property "Footprint" "Connector_JST:JST_XH_B6B-XH-A_1x06_P2.50mm_Vertical" (at 364.49 40.64 0)
+    (property "Footprint" "RCJ2024_kicad_footprints:VL53L0X_VL53L1X_connector" (at 364.49 35.56 0)
       (effects (font (size 1.27 1.27)) hide)
     )
@@
       (effects (font (size 1.27 1.27)) hide)
     )
-    (pin "1")
     (pin "2")
     (pin "3")
@@
     (pin "5")
     (pin "6")
-    (pin "7")
     (instances
       (project "kicad_RCJ"
@@
     )
   )
-  (symbol (lib_id "RCJ_parts:VL53L0X/VL53L1X") (at 364.49 17.78 0) (unit 1)
+  (symbol (lib_id "RCJ_parts:VL53L0X/VL53L1X_NC") (at 364.49 17.78 0) (unit 1)
     (in_bom yes) (on_board yes) (dnp no)
     (property "Reference" "U12" (at 369.57 25.4 0)
@@
       (effects (font (size 1.27 1.27)))
     )
-    (property "Footprint" "Connector_JST:JST_XH_B6B-XH-A_1x06_P2.50mm_Vertical" (at 364.49 17.78 0)
+    (property "Footprint" "RCJ2024_kicad_footprints:VL53L0X_VL53L1X_connector" (at 364.49 12.7 0)
       (effects (font (size 1.27 1.27)) hide)
     )
@@
       (effects (font (size 1.27 1.27)) hide)
     )
-    (pin "1")
     (pin "2")
     (pin "3")
@@
     (pin "5")
     (pin "6")
-    (pin "7")
     (instances
       (project "kicad_RCJ"
@@
     )
   )
-  (symbol (lib_id "RCJ_parts:VL53L0X/VL53L1X") (at 394.97 40.64 0) (unit 1)
+  (symbol (lib_id "RCJ_parts:VL53L0X/VL53L1X_NC") (at 394.97 40.64 0) (unit 1)
     (in_bom yes) (on_board yes) (dnp no)
     (property "Reference" "U16" (at 400.05 48.26 0)
@@
       (effects (font (size 1.27 1.27)))
     )
-    (property "Footprint" "Connector_JST:JST_XH_B6B-XH-A_1x06_P2.50mm_Vertical" (at 394.97 40.64 0)
+    (property "Footprint" "RCJ2024_kicad_footprints:VL53L0X_VL53L1X_connector" (at 394.97 35.56 0)
       (effects (font (size 1.27 1.27)) hide)
     )
@@
       (effects (font (size 1.27 1.27)) hide)
     )
-    (pin "1")
     (pin "2")
     (pin "3")
@@
     (pin "5")
     (pin "6")
-    (pin "7")
     (instances
       (project "kicad_RCJ"
@@
       (effects (font (size 1.27 1.27)) (justify left))
     )
-    (property "Footprint" "" (at 229.362 135.89 90)
+    (property "Footprint" "Resistor_THT:R_Axial_DIN0207_L6.3mm_D2.5mm_P7.62mm_Horizontal" (at 229.362 135.89 90)
       (effects (font (size 1.27 1.27)) hide)
     )
@@
       (effects (font (size 1.27 1.27)) (justify left))
     )
-    (property "Footprint" "" (at 240.792 265.43 90)
+    (property "Footprint" "Resistor_THT:R_Axial_DIN0207_L6.3mm_D2.5mm_P7.62mm_Horizontal" (at 240.792 265.43 90)
       (effects (font (size 1.27 1.27)) hide)
     )
@@
     )
   )
-  (symbol (lib_id "RCJ_parts:VL53L0X/VL53L1X") (at 364.49 63.5 0) (unit 1)
+  (symbol (lib_id "RCJ_parts:VL53L0X/VL53L1X_NC") (at 364.49 63.5 0) (unit 1)
     (in_bom yes) (on_board yes) (dnp no)
     (property "Reference" "U14" (at 369.57 71.12 0)
@@
       (effects (font (size 1.27 1.27)))
     )
-    (property "Footprint" "Connector_JST:JST_XH_B6B-XH-A_1x06_P2.50mm_Vertical" (at 364.49 63.5 0)
+    (property "Footprint" "RCJ2024_kicad_footprints:VL53L0X_VL53L1X_connector" (at 364.49 58.42 0)
       (effects (font (size 1.27 1.27)) hide)
     )
@@
       (effects (font (size 1.27 1.27)) hide)
     )
-    (pin "1")
     (pin "2")
     (pin "3")
@@
     (pin "5")
     (pin "6")
-    (pin "7")
     (instances
       (project "kicad_RCJ"

Commit message: added power delivery to PCB
Parts:
- removed BT1: Battery, symbol Device:Battery
- removed U10, U11, U5, U7, U8, U9: ~, symbol RCJ_parts:XL4015_breakout
- added J23: VBAT_meas_conn, Connector_JST:JST_XH_B2B-XH-A_1x02_P2.50mm_Vertical, symbol Connector_Generic:Conn_01x02
- added J24, J25, J26, J27: Conn_01x02, Connector_JST:JST_XH_B2B-XH-A_1x02_P2.50mm_Vertical, symbol Connector_Generic:Conn_01x02
- added J28: Conn_01x02_5V, Connector_JST:JST_XH_B2B-XH-A_1x02_P2.50mm_Vertical, symbol Connector_Generic:Conn_01x02
- added J29: Conn_01x02_3.3V, Connector_JST:JST_XH_B2B-XH-A_1x02_P2.50mm_Vertical, symbol Connector_Generic:Conn_01x02
Connections:
- net +3.3V: now also J29.2 (Pin_2)
- net +5V: now also J28.2 (Pin_2)
- net GND: now also J23.1 (Pin_1), J24.1 (Pin_1), J25.1 (Pin_1), J26.1 (Pin_1), J27.1 (Pin_1), J28.1 (Pin_1), J29.1 (Pin_1)
- net at J9.1 (Pin_1): now also D4.3 (SIGNAL); no longer D8.2 (SIGNAL)
- net at J9.2 (Pin_2): now also D3.3 (SIGNAL); no longer D7.2 (SIGNAL)
- net at J9.3 (Pin_3): now also D5.3 (SIGNAL); no longer D4.3 (SIGNAL)
- net at J9.4 (Pin_4): now also D6.3 (SIGNAL); no longer D3.3 (SIGNAL)
- net at J9.5 (Pin_5): now also D7.2 (SIGNAL); no longer D5.3 (SIGNAL)
- net at J9.6 (Pin_6): now also D8.2 (SIGNAL); no longer D6.3 (SIGNAL)
- net at R14.1: now also J23.2 (Pin_2)
- net at U3.8 (VIN): now also J26.2 (Pin_2)
- net at U1.8 (VIN): now also J24.2 (Pin_2)
- net at U2.8 (VIN): now also J25.2 (Pin_2)
- net at U4.8 (VIN): now also J27.2 (Pin_2)
Other:
- note removed: "Fuses, switches and voltage measurement?"
- moved on the sheet: J9, R13, R14

Commit message: fixed some connector pin number issues (TOF and colour sensors)
Parts:
- U12, U13, U14, U15, U16, U17, U18, U25: footprint RCJ2024_kicad_footprints:VL53L0X_VL53L1X_connector -> Connector_JST:JST_XH_B5B-XH-A_1x05_P2.50mm_Vertical
- U23: symbol RCJ_parts:adafruit_TCS34725 -> RCJ_parts:adafruit_TCS34725_NC
- U24: symbol RCJ_parts:adafruit_APDS9960 -> RCJ_parts:adafruit_APDS9960_NC
Connections:
- net +3.3V: now also U12.1 (VIN), U13.1 (VIN), U14.1 (VIN), U15.1 (VIN), U16.1 (VIN), U17.1 (VIN), U18.1 (VIN), U23.6 (VIN), U25.1 (VIN); no longer U12.2 (VIN), U13.2 (VIN), U14.2 (VIN), U15.2 (VIN), U16.2 (VIN), U17.2 (VIN), U18.2 (VIN), U23.7 (VIN), U25.2 (VIN)
- net GND: now also U12.2 (GND), U13.2 (GND), U14.2 (GND), U15.2 (GND), U16.2 (GND), U17.2 (GND), U18.2 (GND), U23.5 (GND), U24.2 (GND), U25.2 (GND); no longer U12.3 (GND), U13.3 (GND), U14.3 (GND), U15.3 (GND), U16.3 (GND), U17.3 (GND), U18.3 (GND), U23.6 (GND), U24.3 (GND), U25.3 (GND)
- net SCL: now also U12.4 (SCL), U13.4 (SCL), U14.4 (SCL), U15.4 (SCL), U16.4 (SCL), U17.4 (SCL), U18.4 (SCL), U24.3 (SCL), U25.4 (SCL); no longer U12.5 (SCL), U13.5 (SCL), U14.5 (SCL), U15.5 (SCL), U16.5 (SCL), U17.5 (SCL), U18.5 (SCL), U24.4 (SCL), U25.5 (SCL)
- net SDA: now also U12.3 (SDA), U13.3 (SDA), U14.3 (SDA), U15.3 (SDA), U16.3 (SDA), U17.3 (SDA), U18.3 (SDA), U24.4 (SDA), U25.3 (SDA); no longer U12.4 (SDA), U13.4 (SDA), U14.4 (SDA), U15.4 (SDA), U16.4 (SDA), U17.4 (SDA), U18.4 (SDA), U24.5 (SDA), U25.4 (SDA)
- net at U19.10 (PB1): now also U15.5 (XSHUT); no longer U15.6 (XSHUT)
- net at U19.11 (PB2): now also U13.5 (XSHUT); no longer U13.6 (XSHUT)
- net at U19.12 (PB3): now also U16.5 (XSHUT); no longer U16.6 (XSHUT)
- net at U19.13 (PB4): now also U14.5 (XSHUT); no longer U14.6 (XSHUT)
- net at U19.14 (PB5): now also U17.5 (XSHUT); no longer U17.6 (XSHUT)
- net at U19.15 (PB6): now also U18.5 (XSHUT); no longer U18.6 (XSHUT)
- net at U19.16 (PB7): now also U25.5 (XSHUT); no longer U25.6 (XSHUT)
- net at U19.9 (PB0): now also U12.5 (XSHUT); no longer U12.6 (XSHUT)
- net at J3.1 (Pin_1): now also U24.5 (INT); no longer U24.6 (INT)
- no-connect marks 75 -> 57
Changed lines of the file:
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@@
   (junction (at 77.47 276.86) (diameter 0) (color 0 0 0 0)
   )
-  (no_connect (at 358.14 17.78))
   (no_connect (at 309.88 208.28))
-  (no_connect (at 358.14 55.88))
   (no_connect (at 99.06 127))
   (no_connect (at 350.52 205.74))
   (no_connect (at 320.04 119.38))
   (no_connect (at 330.2 226.06))
-  (no_connect (at 358.14 40.64))
   (no_connect (at 309.88 187.96))
-  (no_connect (at 388.62 99.06))
-  (no_connect (at 388.62 55.88))
   (no_connect (at 350.52 187.96))
   (no_connect (at 309.88 172.72))
@@
   (no_connect (at 309.88 190.5))
   (no_connect (at 210.82 45.72))
-  (no_connect (at 388.62 62.23))
   (no_connect (at 332.74 160.02))
   (no_connect (at 134.62 170.18))
-  (no_connect (at 358.14 33.02))
   (no_connect (at 350.52 210.82))
-  (no_connect (at 358.14 78.74))
   (no_connect (at 327.66 160.02))
-  (no_connect (at 227.33 162.56))
   (no_connect (at 350.52 180.34))
   (no_connect (at 335.28 160.02))
@@
   (no_connect (at 327.66 226.06))
   (no_connect (at 309.88 170.18))
-  (no_connect (at 252.73 162.56))
   (no_connect (at 350.52 185.42))
   (no_connect (at 325.12 226.06))
-  (no_connect (at 358.14 102.87))
   (no_connect (at 99.06 85.09))
-  (no_connect (at 358.14 87.63))
-  (no_connect (at 358.14 63.5))
   (no_connect (at 309.88 180.34))
   (no_connect (at 350.52 195.58))
   (no_connect (at 257.81 209.55))
   (no_connect (at 332.74 226.06))
-  (no_connect (at 388.62 77.47))
   (no_connect (at 180.34 172.72))
   (no_connect (at 99.06 168.91))
   (no_connect (at 335.28 226.06))
-  (no_connect (at 388.62 34.29))
   (no_connect (at 332.74 119.38))
   (no_connect (at 311.15 63.5))
@@
   (no_connect (at 325.12 160.02))
   (no_connect (at 350.52 198.12))
-  (no_connect (at 388.62 83.82))
   (no_connect (at 309.88 198.12))
   (no_connect (at 350.52 200.66))
@@
   (no_connect (at 350.52 203.2))
   (no_connect (at 308.61 63.5))
-  (no_connect (at 388.62 19.05))
   (no_connect (at 210.82 73.66))
   (no_connect (at 309.88 200.66))
-  (no_connect (at 388.62 40.64))
   (wire (pts (xy 99.06 66.04) (xy 99.06 69.85))
     (stroke (width 0) (type default))
@@
       (effects (font (size 1.27 1.27)))
     )
-    (property "Footprint" "RCJ2024_kicad_footprints:VL53L0X_VL53L1X_connector" (at 394.97 78.74 0)
+    (property "Footprint" "Connector_JST:JST_XH_B5B-XH-A_1x05_P2.50mm_Vertical" (at 394.97 78.74 0)
       (effects (font (size 1.27 1.27)) hide)
     )
@@
     (pin "4")
     (pin "5")
-    (pin "6")
+    (pin "1")
     (instances
       (project "kicad_RCJ"
@@
     )
   )
-  (symbol (lib_id "RCJ_parts:adafruit_TCS34725") (at 225.425 154.94 0) (unit 1)
+  (symbol (lib_id "RCJ_parts:adafruit_TCS34725_NC") (at 225.425 154.94 0) (unit 1)
     (in_bom yes) (on_board yes) (dnp no)
     (property "Reference" "U23" (at 224.79 151.13 0)
@@
     (pin "5")
     (pin "6")
-    (pin "7")
     (instances
       (project "kicad_RCJ"
@@
       (effects (font (size 1.27 1.27)))
     )
-    (property "Footprint" "RCJ2024_kicad_footprints:VL53L0X_VL53L1X_connector" (at 394.97 57.15 0)
+    (property "Footprint" "Connector_JST:JST_XH_B5B-XH-A_1x05_P2.50mm_Vertical" (at 394.97 57.15 0)
       (effects (font (size 1.27 1.27)) hide)
     )
@@
     (pin "4")
     (pin "5")
-    (pin "6")
+    (pin "1")
     (instances
       (project "kicad_RCJ"
@@
     )
   )
-  (symbol (lib_id "RCJ_parts:adafruit_APDS9960") (at 254 154.94 0) (unit 1)
+  (symbol (lib_id "RCJ_parts:adafruit_APDS9960_NC") (at 254 154.94 0) (unit 1)
     (in_bom yes) (on_board yes) (dnp no)
     (property "Reference" "U24" (at 254 151.13 0)
@@
     (pin "4")
     (pin "5")
-    (pin "6")
     (instances
       (project "kicad_RCJ"
@@
       (effects (font (size 1.27 1.27)))
     )
-    (property "Footprint" "RCJ2024_kicad_footprints:VL53L0X_VL53L1X_connector" (at 394.97 13.97 0)
+    (property "Footprint" "Connector_JST:JST_XH_B5B-XH-A_1x05_P2.50mm_Vertical" (at 394.97 13.97 0)
       (effects (font (size 1.27 1.27)) hide)
     )
@@
     (pin "4")
     (pin "5")
-    (pin "6")
+    (pin "1")
     (instances
       (project "kicad_RCJ"
@@
       (effects (font (size 1.27 1.27)))
     )
-    (property "Footprint" "RCJ2024_kicad_footprints:VL53L0X_VL53L1X_connector" (at 364.49 82.55 0)
+    (property "Footprint" "Connector_JST:JST_XH_B5B-XH-A_1x05_P2.50mm_Vertical" (at 364.49 82.55 0)
       (effects (font (size 1.27 1.27)) hide)
     )
@@
     (pin "4")
     (pin "5")
-    (pin "6")
+    (pin "1")
     (instances
       (project "kicad_RCJ"
@@
       (effects (font (size 1.27 1.27)))
     )
-    (property "Footprint" "RCJ2024_kicad_footprints:VL53L0X_VL53L1X_connector" (at 364.49 35.56 0)
+    (property "Footprint" "Connector_JST:JST_XH_B5B-XH-A_1x05_P2.50mm_Vertical" (at 364.49 35.56 0)
       (effects (font (size 1.27 1.27)) hide)
     )
@@
     (pin "4")
     (pin "5")
-    (pin "6")
+    (pin "1")
     (instances
       (project "kicad_RCJ"
@@
       (effects (font (size 1.27 1.27)))
     )
-    (property "Footprint" "RCJ2024_kicad_footprints:VL53L0X_VL53L1X_connector" (at 364.49 12.7 0)
+    (property "Footprint" "Connector_JST:JST_XH_B5B-XH-A_1x05_P2.50mm_Vertical" (at 364.49 12.7 0)
       (effects (font (size 1.27 1.27)) hide)
     )
@@
     (pin "4")
     (pin "5")
-    (pin "6")
+    (pin "1")
     (instances
       (project "kicad_RCJ"
@@
       (effects (font (size 1.27 1.27)))
     )
-    (property "Footprint" "RCJ2024_kicad_footprints:VL53L0X_VL53L1X_connector" (at 394.97 35.56 0)
+    (property "Footprint" "Connector_JST:JST_XH_B5B-XH-A_1x05_P2.50mm_Vertical" (at 394.97 35.56 0)
       (effects (font (size 1.27 1.27)) hide)
     )
@@
     (pin "4")
     (pin "5")
-    (pin "6")
+    (pin "1")
     (instances
       (project "kicad_RCJ"
@@
       (effects (font (size 1.27 1.27)))
     )
-    (property "Footprint" "RCJ2024_kicad_footprints:VL53L0X_VL53L1X_connector" (at 364.49 58.42 0)
+    (property "Footprint" "Connector_JST:JST_XH_B5B-XH-A_1x05_P2.50mm_Vertical" (at 364.49 58.42 0)
       (effects (font (size 1.27 1.27)) hide)
     )
@@
     (pin "4")
     (pin "5")
-    (pin "6")
+    (pin "1")
     (instances
       (project "kicad_RCJ"
@@
   )
   (symbol (lib_id "Connector:Raspberry_Pi_2_3") (at 330.2 193.04 0) (unit 1)
-    (in_bom yes) (on_board yes) (dnp no) (fields_autoplaced)
+    (in_bom yes) (on_board no) (dnp no) (fields_autoplaced)
     (property "Reference" "J1" (at 337.4741 157.48 0)
       (effects (font (size 1.27 1.27)) (justify left))
